Commit message: Update robot dimensions: wheel_base=95mm, lidar=55mm/130mm, robot_radius=0.14m

File: my_4wd_robot.urdf (robot description, URDF)
Before this commit: robot my_4wd_robot, 6 links, 5 joints
Links:
- link base_laser: geometry collision cylinder length=0.04 radius=0.035; visual cylinder length=0.04 radius=0.035
- link base_link: geometry collision box size=0.200 0.200 0.095; visual box size=0.200 0.200 0.095
- link front_left_wheel: geometry collision cylinder length=0.03 radius=0.04; visual cylinder length=0.03 radius=0.04
- link front_right_wheel: geometry collision cylinder length=0.03 radius=0.04; visual cylinder length=0.03 radius=0.04
- link rear_left_wheel: geometry collision cylinder length=0.03 radius=0.04; visual cylinder length=0.03 radius=0.04
- link rear_right_wheel: geometry collision cylinder length=0.03 radius=0.04; visual cylinder length=0.03 radius=0.04
Joints:
- joint front_left_joint: origin xyz=0.1 0.12 -0.04 rpy=1.5708 0 0 -> xyz=0.075 0.0625 -0.0075 rpy=1.5708 0 0
- joint front_right_joint: origin xyz=0.1 -0.12 -0.04 rpy=1.5708 0 0 -> xyz=0.075 -0.0625 -0.0075 rpy=1.5708 0 0
- joint laser_joint: origin xyz=0.012548 0 0.08 rpy=0 0 0 -> xyz=0.055 0 0.130 rpy=0 0 0
- joint rear_left_joint: origin xyz=-0.1 0.12 -0.04 rpy=1.5708 0 0 -> xyz=-0.075 0.0625 -0.0075 rpy=1.5708 0 0
- joint rear_right_joint: origin xyz=-0.1 -0.12 -0.04 rpy=1.5708 0 0 -> xyz=-0.075 -0.0625 -0.0075 rpy=1.5708 0 0
